File: PCBs/GroundPCB/GroundPCB.kicad_sch (KiCad schematic)
At the start: 67 parts, among them IC1 SWITCH-HSWA4-63DR+, IC2 SWITCH-HSWA4-63DR+, J1 SMA-LPRS-CONNECTOR, J2 Conn_01x04, J3 Conn_01x04, SW1 SW_SPST, U1 HMC452ST89ETR, U2 PGA-103+, U3 RFM96W-433S2, U4 DS3231M

Commit message: post-review revisions
Parts:
- C13: value 10u -> 1u
- C14: value 0.1u -> 100n
- C15, C16: value 100p -> 100n
- C19, C20: value 0.47u -> 100n
- C2, C5: value 0.01u -> 10n
- C7: value 0.33u -> 330n
Changed lines of the file:
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@@
   (title_block
     (title "NARWAL")
-    (date "2022-11-13")
+    (date "2022-11-19")
     (rev "1")
     (company "Rice Eclipse")
+    (comment 1 "RF Communications")
   )
   (junction (at 109.22 196.85) (diameter 0) (color 0 0 0 0)
@@
       (effects (font (size 1.27 1.27)) (justify left))
     )
-    (property "Value" "100p" (id 1) (at 213.36 186.055 0)
+    (property "Value" "100n" (id 1) (at 213.36 186.055 0)
       (effects (font (size 1.27 1.27)) (justify left))
     )
@@
     (in_bom yes) (on_board yes)
     (property "Reference" "C14" (id 0) (at 209.55 60.96 90))
-    (property "Value" "0.1u" (id 1) (at 209.55 63.5 90))
+    (property "Value" "100n" (id 1) (at 209.55 63.5 90))
     (property "Footprint" "Capacitor_SMD:C_1206_3216Metric" (id 2) (at 213.36 56.1848 0)
       (effects (font (size 1.27 1.27)) hide)
@@
     (in_bom yes) (on_board yes)
     (property "Reference" "C2" (id 0) (at 82.55 222.25 90))
-    (property "Value" "0.01u" (id 1) (at 82.55 224.79 90))
+    (property "Value" "10n" (id 1) (at 82.55 224.79 90))
     (property "Footprint" "Capacitor_SMD:C_1206_3216Metric" (id 2) (at 86.36 227.6348 0)
       (effects (font (size 1.27 1.27)) hide)
@@
     (in_bom yes) (on_board yes)
     (property "Reference" "C19" (id 0) (at 321.31 50.8 90))
-    (property "Value" "0.47u" (id 1) (at 321.31 53.34 90))
+    (property "Value" "100n" (id 1) (at 321.31 53.34 90))
     (property "Footprint" "Capacitor_SMD:C_1206_3216Metric" (id 2) (at 325.12 56.1848 0)
       (effects (font (size 1.27 1.27)) hide)
@@
     (in_bom yes) (on_board yes)
     (property "Reference" "C5" (id 0) (at 113.03 222.25 90))
-    (property "Value" "0.01u" (id 1) (at 113.03 224.79 90))
+    (property "Value" "10n" (id 1) (at 113.03 224.79 90))
     (property "Footprint" "Capacitor_SMD:C_1206_3216Metric" (id 2) (at 116.84 227.6348 0)
       (effects (font (size 1.27 1.27)) hide)
@@
   (symbol (lib_id "Device:C") (at 342.9 54.61 0) (unit 1)
     (in_bom yes) (on_board yes)
-    (property "Reference" "C20" (id 0) (at 346.71 54.61 0))
-    (property "Value" "0.47u" (id 1) (at 346.71 57.15 0))
+    (property "Reference" "C20" (id 0) (at 347.345 54.61 0))
+    (property "Value" "100n" (id 1) (at 347.345 57.15 0))
     (property "Footprint" "Capacitor_SMD:C_1206_3216Metric" (id 2) (at 343.8652 58.42 0)
       (effects (font (size 1.27 1.27)) hide)
@@
   (symbol (lib_id "Connector:TestPoint_Small") (at 223.52 177.8 90) (unit 1)
     (in_bom yes) (on_board yes)
-    (property "Reference" "TP13" (id 0) (at 225.425 175.895 90)
+    (property "Reference" "TP13" (id 0) (at 226.695 175.895 90)
       (effects (font (size 1.27 1.27)) (justify left))
     )
@@
     (in_bom yes) (on_board yes)
     (property "Reference" "C7" (id 0) (at 115.57 207.01 90))
-    (property "Value" "0.33u" (id 1) (at 115.57 209.55 90))
+    (property "Value" "330n" (id 1) (at 115.57 209.55 90))
     (property "Footprint" "Capacitor_SMD:C_1206_3216Metric" (id 2) (at 119.38 202.2348 0)
       (effects (font (size 1.27 1.27)) hide)
@@
     (in_bom yes) (on_board yes)
     (property "Reference" "C13" (id 0) (at 209.55 44.45 90))
-    (property "Value" "10u" (id 1) (at 209.55 46.99 90))
+    (property "Value" "1u" (id 1) (at 209.55 46.99 90))
     (property "Footprint" "Capacitor_SMD:C_1206_3216Metric" (id 2) (at 213.36 49.8348 0)
       (effects (font (size 1.27 1.27)) hide)
@@
       (effects (font (size 1.27 1.27)) (justify left))
     )
-    (property "Value" "100p" (id 1) (at 213.36 262.255 0)
+    (property "Value" "100n" (id 1) (at 213.36 262.255 0)
       (effects (font (size 1.27 1.27)) (justify left))
     )
@@
     )
     (path "/17650cc2-0ea9-4df9-8435-fe0eea675be7"
-      (reference "C2") (unit 1) (value "0.01u") (footprint "Capacitor_SMD:C_1206_3216Metric")
+      (reference "C2") (unit 1) (value "10n") (footprint "Capacitor_SMD:C_1206_3216Metric")
     )
     (path "/a53ab678-9dec-4b70-b8b1-2aa2dacdddd3"
@@
     )
     (path "/2ae17081-2113-4170-b77b-dd0f8e7a72d2"
-      (reference "C5") (unit 1) (value "0.01u") (footprint "Capacitor_SMD:C_1206_3216Metric")
+      (reference "C5") (unit 1) (value "10n") (footprint "Capacitor_SMD:C_1206_3216Metric")
     )
     (path "/19b0f565-747f-463b-a462-59a985266175"
@@
     )
     (path "/91caf652-ecda-4df6-8747-017e460ff584"
-      (reference "C7") (unit 1) (value "0.33u") (footprint "Capacitor_SMD:C_1206_3216Metric")
+      (reference "C7") (unit 1) (value "330n") (footprint "Capacitor_SMD:C_1206_3216Metric")
     )
     (path "/059c0705-8396-4665-8988-e0cc5b143c95"
@@
     )
     (path "/b6f34181-b7d9-4664-9f3e-6973737275df"
-      (reference "C13") (unit 1) (value "10u") (footprint "Capacitor_SMD:C_1206_3216Metric")
+      (reference "C13") (unit 1) (value "1u") (footprint "Capacitor_SMD:C_1206_3216Metric")
     )
     (path "/0e209cfa-c7fe-4d64-88d9-c26302a40471"
-      (reference "C14") (unit 1) (value "0.1u") (footprint "Capacitor_SMD:C_1206_3216Metric")
+      (reference "C14") (unit 1) (value "100n") (footprint "Capacitor_SMD:C_1206_3216Metric")
     )
     (path "/01a936b3-6c38-4036-8b76-f79360849d4a"
-      (reference "C15") (unit 1) (value "100p") (footprint "Capacitor_SMD:C_1206_3216Metric")
+      (reference "C15") (unit 1) (value "100n") (footprint "Capacitor_SMD:C_1206_3216Metric")
     )
     (path "/c3084e0e-e25f-430e-8bff-d9f3cf062131"
-      (reference "C16") (unit 1) (value "100p") (footprint "Capacitor_SMD:C_1206_3216Metric")
+      (reference "C16") (unit 1) (value "100n") (footprint "Capacitor_SMD:C_1206_3216Metric")
     )
     (path "/f83e5b05-ee89-4771-b336-a7e53757239c"
@@
     )
     (path "/1ae219e9-8d6d-4f2f-b8ad-7abb68ff887e"
-      (reference "C19") (unit 1) (value "0.47u") (footprint "Capacitor_SMD:C_1206_3216Metric")
+      (reference "C19") (unit 1) (value "100n") (footprint "Capacitor_SMD:C_1206_3216Metric")
     )
     (path "/56498129-9393-4382-9cef-d7785e68e019"
-      (reference "C20") (unit 1) (value "0.47u") (footprint "Capacitor_SMD:C_1206_3216Metric")
+      (reference "C20") (unit 1) (value "100n") (footprint "Capacitor_SMD:C_1206_3216Metric")
     )
     (path "/638bb3ce-2ece-4bf6-8f0d-a5a1cf43d309"
